Commit message: Add files via upload

File: multiple_robots/description/robot4_diff_bot.urdf (robot description, URDF)
Before this commit: robot robot1_swerve_bot, 5 links, 4 joints
Links:
- link base_link: geometry collision mesh filename=package://multiple_robots/meshes/Frame_DIFF.STL; visual mesh filename=package://multiple_robots/meshes/Frame_DIFF.STL
Joints:
- joint lidar_joint: origin xyz=0.2555 0 0.05 rpy=0.0 0.0 0.0 -> xyz=0.15 0 0.1406 rpy=0.0 0.0 0.0
