Commit message: Add files via upload

File: multiple_robots/description/robot1_swerve_bot.urdf (robot description, URDF)
Before this commit: robot robot1_swerve_bot, 5 links, 4 joints
Joints:
- joint numb_joint: origin xyz=0 0 0.1206 -> xyz=0 0 0.1106

File: multiple_robots/description/robot2_swerve_bot.urdf (robot description, URDF)
Before this commit: robot robot2_swerve_bot, 5 links, 4 joints
Joints:
- joint numb_joint: origin xyz=0 0 0.1206 -> xyz=0 0 0.1106

File: multiple_robots/description/robot3_swerve_bot.urdf (robot description, URDF)
Before this commit: robot robot3_swerve_bot, 5 links, 4 joints
Joints:
- joint numb_joint: origin xyz=0 0 0.1206 -> xyz=0 0 0.1106

File: multiple_robots/description/robot4_diff_bot.urdf (robot description, URDF)
Before this commit: robot robot4_diff_bot, 5 links, 4 joints
Joints:
- joint numb_joint: origin xyz=0 0 0.1206 -> xyz=0 0 0.1106
