Commit message: Add files via upload

File: multiple_robots/description/robot5_diff_bot.urdf (robot description, URDF)
Before this commit: robot robot4_diff_bot, 5 links, 4 joints
Links:
- link numb_link: geometry collision mesh filename=package://multiple_robots/meshes/Numb_5.STL; visual mesh filename=package://multiple_robots/meshes/Numb_5.STL

File: multiple_robots/description/robot6_diff_bot.urdf (robot description, URDF)
Before this commit: robot robot4_diff_bot, 5 links, 4 joints
Links:
- link numb_link: geometry collision mesh filename=package://multiple_robots/meshes/Numb_6.STL; visual mesh filename=package://multiple_robots/meshes/Numb_6.STL
